File: electronic/RevA/mfi.kicad_sch (KiCad schematic)
At the start: 17 parts, among them J1 RPi_GPIO, J4 TYPE-C-31-M-12, U1 MFI343S00177, U2 MFI337S3959, U3 MFI343S00177

Commit message: Add note to schematic
Other:
- note added: "External power for Rpi"
- note added: "I2C Addr 0x10"
- note added: "I2C Addr 0x11"
- note removed: "Rpi power in from USB-C"
Changed lines of the file:
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@@
 		(company "Signalius")
 	)
-	(text "Rpi power in from USB-C\n"
+	(text "I2C Addr\n0x10"
 		(exclude_from_sim no)
-		(at 24.13 25.146 90)
+		(at 59.69 94.996 0)
 		(effects
 			(font
+				(size 1.27 1.27)
+			)
+		)
+	)
+	(text "I2C Addr\n0x11"
+		(exclude_from_sim no)
+		(at 57.15 121.412 0)
+		(effects
+			(font
+				(size 1.27 1.27)
+			)
+		)
+	)
+	(text "External power for Rpi\n"
+		(exclude_from_sim no)
+		(at 26.162 25.654 90)
+		(effects
+			(font
